Commit message: Remove everything except the description and gazebo plugins packages. Update the readme

File: ouster_description/urdf/OS1-64.urdf.xacro (robot description, xacro)
@@ -6,5 +6,31 @@
       <xacro:insert_block name="origin" />
       <parent link="${parent}"/>
+      <child link="${name}_base_link"/>
+    </joint>
+    <link name="${name}_base_link" />
+    <joint name="${name}_base_to_baseplate" type="fixed">
+      <parent link="${name}_base_link"/>
+      <child link="${name}_baseplate" />
+      <origin xyz="0 0 0.008"/>
+    </joint>
+    <link name="${name}_baseplate">
+      <visual>
+        <geometry>
+          <box size="0.112 0.112 0.016" />
+        </geometry>
+        <material name="silver">
+          <color rgba="0.5 0.5 0.5 1.0" />
+        </material>
+      </visual>
+      <collision>
+        <geometry>
+          <box size="0.112 0.112 0.016" />
+        </geometry>
+      </collision>
+    </link>
+    <joint name="${name}_baseplate_to_body" type="fixed">
+      <parent link="${name}_baseplate"/>
       <child link="${name}"/>
+      <origin xyz="0 0 0.042" rpy="0 0 0" />
     </joint>
     <link name="${name}">

Commit message: Update topic names and frame/link names to match ouster ROS driver

File: ouster_description/urdf/OS1-64.urdf.xacro (robot description, xacro)
@@ -2,5 +2,5 @@
 <robot xmlns:xacro="http://www.ros.org/wiki/xacro" name="OS1-64">
   <xacro:property name="M_PI" value="3.1415926535897931" />
-  <xacro:macro name="OS1-64" params="*origin parent:=base_link name:=os1_sensor topic_points:=/os1_cloud_node/points topic_imu:=/os1_cloud_node/imu hz:=10 lasers:=64 samples:=512 min_range:=0.9 max_range:=75.0 noise:=0.008 min_angle:=-${M_PI} max_angle:=${M_PI} lidar_link:=os1_lidar imu_link:=os1_imu vfov_min:=-.26 vfov_max:=.26">
+  <xacro:macro name="OS1-64" params="*origin parent:=base_link name:=os_sensor topic_points:=/ouster/points topic_imu:=/ouster/imu hz:=10 lasers:=64 samples:=512 min_range:=0.9 max_range:=75.0 noise:=0.008 min_angle:=-${M_PI} max_angle:=${M_PI} lidar_link:=os_lidar imu_link:=os_imu vfov_min:=-.26 vfov_max:=.26">
     <joint name="${name}_mount_joint" type="fixed">
       <xacro:insert_block name="origin" />
